File: hardware/mcu_board/mcu_board.kicad_sch (KiCad schematic)
At the start: 0 parts

Commit message: PCB  first commits
Parts:
- added J1: Conn_01x06_Pin, Connector_PinHeader_1.00mm:PinHeader_1x06_P1.00mm_Horizontal, symbol Connector:Conn_01x06_Pin
- added J2: Conn_01x04_Pin, Connector_PinHeader_1.00mm:PinHeader_1x04_P1.00mm_Horizontal, symbol Connector:Conn_01x04_Pin
Connections:
- new net Vertical axis: J1.1 (Pin_1)
- new net horizontal_axis: J2.3 (Pin_3)
- new net horizontalaxis: J1.2 (Pin_2)
- new net jaw_bottom: J2.2 (Pin_2)
- new net jaw_upper: J2.1 (Pin_1)
- new net left_bottom: J1.6 (Pin_6)
- new net left_upper: J1.5 (Pin_5)
- new net right_bottom: J1.4 (Pin_4)
- new net right_upper: J1.3 (Pin_3)
- new net vertical_axis: J2.4 (Pin_4)
Other:
- note added: "eyes servomotors"
- note added: "head servomotors"
