File: hardware/eyes/eyes.kicad_sch (KiCad schematic)
At the start: 10 parts, among them J1 Conn_01x09_Pin, J2 Conn_01x09_Pin, J3 Conn_01x09_Pin, J4 Conn_01x09_Pin, J5 Barrel_Jack, J8 Conn_01x22, J9 Conn_01x22

Commit message: Finishing eyes PCB and exporting BOM
Parts:
- J5: footprint Connector_BarrelJack:BarrelJack_SwitchcraftConxall_RAPC10U_Horizontal -> Connector_BarrelJack:BarrelJack_Horizontal
Connections:
- no-connect marks 8 -> 6
Changed lines of the file:
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@@
-	)
-	(no_connect
-		(at 213.36 43.18)
 	)
 	(no_connect
@@
 	(no_connect
 		(at 180.34 92.71)
-	)
-	(no_connect
-		(at 222.25 64.77)
 	)
 	(wire
@@
 			)
 		)
-		(property "Footprint" "Connector_BarrelJack:BarrelJack_SwitchcraftConxall_RAPC10U_Horizontal"
+		(property "Footprint" "Connector_BarrelJack:BarrelJack_Horizontal"
 			(at 223.52 63.246 0)
 			(hide yes)
