File: hardware/stm/stm.kicad_sch (KiCad schematic)
At the start: 1 part, among them U1 STM32F103C8Tx

Commit message: Working on STM32 schematic
Parts:
- removed U1: STM32F103C8Tx, Package_QFP:LQFP-48_7x7mm_P0.5mm, symbol MCU_ST_STM32F1:STM32F103C8Tx
- added C1, C2: 0.1uF, symbol Device:C
- added R2, R3: R, symbol Device:R
- added U1: STM32L476RGTx, Package_QFP:LQFP-64_10x10mm_P0.5mm, symbol MCU_ST_STM32L4:STM32L476RGTx
- added U2: LSM6DS3, Package_LGA:LGA-14_3x2.5mm_P0.5mm_LayoutBorder3x4y, symbol Sensor_Motion:LSM6DS3
Connections:
- new net: U1.18 (VSS), U1.31 (VSS), U1.47 (VSS), U1.63 (VSS)
- new net +3V3: C1.2, C2.1, R2.1, R3.1, U1.19 (VDD), U2.12 (CS), U2.5 (VDDIO), U2.8 (VDD)
- new net GND: C1.1, C2.2, U1.12 (VSSA), U2.1 (SDO/SA0), U2.2 (SDX), U2.3 (SCX), U2.6 (GND), U2.7 (GND)
- new net GYRO_INT1: U2.4 (INT1)
- new net GYRO_INT2: U2.9 (INT2)
- new net HEAD_HORIZONTAL_PWM: U1.22 (PA6)
- new net HEAD_VERTICAL_PWM: U1.23 (PA7)
- new net LEFT_PUPIL_PWM: U1.14 (PA0)
- new net LOWER_JAW_PWM: U1.27 (PB1)
- new net RESET: U1.7 (NRST)
- new net RIGHT_PUPIL_PWM: U1.15 (PA1)
- new net SCL: R3.2, U2.13 (SCL)
- new net SDA: R2.2, U2.14 (SDA)
- new net UART_RX: U1.17 (PA3)
- new net UART_TX: U1.16 (PA2)
- new net UPPER_JAW_PWM: U1.26 (PB0)
- no-connect marks 0 -> 3
Other:
- note added: "0x6A"
- note added: "GYROSCOPE/ACCELEROMETER"
- note added: "MCU"
